Commit message: Toki's changes

File: resources/kuka_iiwa/kuka_iiwa.urdf (robot description, URDF)
Before this commit: robot kuka_iiwa, 8 links, 7 joints
Links:
- link base_link: geometry collision mesh filename=meshes/base.obj scale=1 1 1; visual mesh filename=meshes/base.obj scale=1 1 1
- link link0: geometry collision mesh filename=meshes/link0.obj scale=1 1 1; visual mesh filename=meshes/link0.obj scale=1 1 1
- link link1: geometry collision mesh filename=meshes/link1.obj scale=1 1 1; visual mesh filename=meshes/link1.obj scale=1 1 1
- link link2: geometry collision mesh filename=meshes/link2.obj scale=1 1 1; visual mesh filename=meshes/link2.obj scale=1 1 1
- link link3: geometry collision mesh filename=meshes/link3.obj scale=1 1 1; visual mesh filename=meshes/link3.obj scale=1 1 1
- link link4: geometry collision mesh filename=meshes/link4.obj scale=1 1 1; visual mesh filename=meshes/link4.obj scale=1 1 1
- link link5: geometry collision mesh filename=meshes/link5.obj scale=1 1 1; visual mesh filename=meshes/link5.obj scale=1 1 1
- link link6: geometry collision cylinder length=0.02 radius=0.05; collision mesh filename=meshes/link6.obj scale=1 1 1
