Commit message: Urdfs

File: src/pp_project/kuka_iiwa_pp.urdf (robot description, URDF)
Before this commit: robot kuka_iiwa, 8 links, 7 joints
Links:
- link link6: geometry collision box size=0.33 0.33 0.02; visual box size=0.33 0.33 0.02

Commit message: Almost works but can't quite get to the desired joint space

File: src/pp_project/kuka_iiwa_pp.urdf (robot description, URDF)
Before this commit: robot kuka_iiwa, 8 links, 7 joints
Links:
- link link6: geometry visual mesh filename=kuka_iiwa_graphics/link6.obj scale=1 1 1

Commit message: update

File: src/pp_project/kuka_iiwa_pp.urdf (robot description, URDF)
Before this commit: robot kuka_iiwa, 8 links, 7 joints
Links:
- link base_link: geometry collision mesh filename=kuka_iiwa_graphics/base.obj scale=1 1 1; visual mesh filename=kuka_iiwa_graphics/base.obj scale=1 1 1
- link link0: geometry collision mesh filename=kuka_iiwa_graphics/link0.obj scale=1 1 1; visual mesh filename=kuka_iiwa_graphics/link0.obj scale=1 1 1
- link link1: geometry collision mesh filename=kuka_iiwa_graphics/link1.obj scale=1 1 1; visual mesh filename=kuka_iiwa_graphics/link1.obj scale=1 1 1
- link link2: geometry collision mesh filename=kuka_iiwa_graphics/link2.obj scale=1 1 1; visual mesh filename=kuka_iiwa_graphics/link2.obj scale=1 1 1
- link link3: geometry collision mesh filename=kuka_iiwa_graphics/link3.obj scale=1 1 1; visual mesh filename=kuka_iiwa_graphics/link3.obj scale=1 1 1
- link link4: geometry collision mesh filename=kuka_iiwa_graphics/link4.obj scale=1 1 1; visual mesh filename=kuka_iiwa_graphics/link4.obj scale=1 1 1
- link link5: geometry collision mesh filename=kuka_iiwa_graphics/link5.obj scale=1 1 1; visual mesh filename=kuka_iiwa_graphics/link5.obj scale=1 1 1

Commit message: Latest changes

File: src/pp_project/kuka_iiwa_pp.urdf (robot description, URDF)
Before this commit: robot kuka_iiwa, 8 links, 7 joints
Links:
- link link6: geometry collision box size=0.33 0.33 0.02; collision mesh filename=kuka_iiwa_graphics/link6.obj scale=1 1 1
